File: ThermalSensorsDriver.kicad_sch (KiCad schematic)
At the start: 35 parts, among them J201 Conn_02x12_Odd_Even, U201 LTC2983

Commit message: Fixes issues from revision 1.0
Signed-off-by: Alexis Jeandet <alexis.jeandet@member.fsf.org>
Other:
- company: (none) -> LPP/CNRS
Changed lines of the file:
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@@
 (kicad_sch (version 20211123) (generator eeschema)
   (paper "A4")
+  (title_block
+    (date "2023-02-07")
+    (rev "1.1")
+    (company "LPP/CNRS")
+  )
   (junction (at 69.85 70.485) (diameter 0) (color 0 0 0 0)
   )
@@
   (symbol (lib_id "power:GND") (at 73.66 70.485 90) (unit 1)
     (in_bom yes) (on_board yes) (fields_autoplaced)
-    (property "Reference" "#PWR?" (id 0) (at 80.01 70.485 0)
-      (effects (font (size 1.27 1.27)) hide)
-    )
+    (property "Reference" "#PWR0122" (id 0) (at 80.01 70.485 0)
+      (effects (font (size 1.27 1.27)) hide)
+    )
