File: ThermalSensorsDriver.kicad_sch (KiCad schematic)
At the start: 35 parts, among them J201 Conn_02x12_Odd_Even, U201 LTC2983

Commit message: 1.0 release
Signed-off-by: Alexis Jeandet <alexis.jeandet@member.fsf.org>
Other:
- company: (none) -> Laboratory of Plasma Physics
- title: (none) -> Thermomix
Changed lines of the file:
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@@
 (kicad_sch (version 20211123) (generator eeschema)
   (paper "A4")
+  (title_block
+    (title "Thermomix")
+    (date "2022-06-03")
+    (rev "1.0")
+    (company "Laboratory of Plasma Physics")
+    (comment 1 "Alexis Jeandet <alexis.jeandet@member.fsf.org>")
+  )
   (junction (at 69.85 70.485) (diameter 0) (color 0 0 0 0)
   )
